File: Harness_DIY_Engine_monitoring-06/outputs.kicad_sch (KiCad schematic)
At the start: 32 parts, among them J1 Conn_01x10_Pin, J10 Conn_01x02_Socket, J14 Conn_01x02_Socket, J15 Conn_01x02_Pin, J2 Conn_01x10_Socket, J3 Conn_01x04, J4 Conn_01x04_Socket, J5 Conn_01x02_Socket, J6 Conn_01x02_Pin, J7 Conn_01x02_Pin, J8 Conn_01x02_Socket, J9 Conn_01x02_Pin, K1 Relay_SPDT, K2 Relay_SPDT, K3 Relay_SPDT, U10 ac_lp, U11 Nextion-Touchscreen, U2 FreematicsOBD-II_I2C, U3 Conn,Deutsh_DT-6F, U4 Conn,Deutsh_DT-6M, U5 Con_GT-150-12_M, U6 Driver_DC_BTN8982, U7 Driver_DC_BTN8982

Commit message: Many calibrations made
Still early days of getting code fixes and analog inputs calibrated
Other:
- title: Tahoe_md_wiring -> Harness_DIY_Engine_monitoring
Changed lines of the file:
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@@
 	(paper "USLetter")
 	(title_block
-		(title "Tahoe_md_wiring")
-		(date "2024-12-08")
-		(rev "0.3")
+		(title "Harness_DIY_Engine_monitoring")
+		(date "2024-12-19")
+		(rev "0.6")
 		(comment 1 "Wiring harness & power driver schematic")
-		(comment 2 "Pairs with Tahoe_mb versioson 0.4 & 0.5")
+		(comment 2 "Pairs with PCB_DIY_Engine_Monitoring")
 	)
 	(junction
